File: ControlBoard/CDFR2027-PAMIs-ELEC-control.kicad_pcb (KiCad board)
At the start: 4 copper layers, 81 parts, among them Q1 PMOS

Commit message: Feat: multiplex power over usb + add gitignore
Parts:
- added D1: D_Schottky, Diode_SMD:D_0603_1608Metric, F.Cu at (187.3, 78.5)
- added D2: D_Schottky, Diode_SMD:D_0603_1608Metric, F.Cu at (187.3, 81.1)
- added R23: 470, Resistor_SMD:R_0603_1608Metric, F.Cu at (193.5, 78.5)
- added USB1: LED, Diode_SMD:D_0603_1608Metric, F.Cu at (193.5, 82.8)
- R20: value 5.1k -> 200; footprint Resistor_SMD:R_0603_1608Metric -> Resistor_SMD:R_0603_1608Metric_Pad0.98x0.95mm_HandSolder
- R22: value 470 -> 5.1k
- USB_C1: footprint Connector_USB:USB_C_Receptacle_G-Switch_GT-USB-7051x -> Connector_USB:USB_C_Receptacle_GCT_USB4105-xx-A_16P_TopMnt_Horizontal
- moved JP2 163.4 mm to (105.5, 74.0), turned to 90 degrees
- moved LDO1 157.5 mm to (106.5, 80.1), turned to 90 degrees
- moved C10 155.2 mm to (105.5, 85.1), turned to 90 degrees
- moved C11 152.1 mm to (108.0, 85.1), turned to 90 degrees
- moved SW_ENABLE1 139.4 mm to (151.0, 89.0)
- moved R1 136.2 mm to (152.8, 83.2), turned to 90 degrees
- moved R2 132.6 mm to (150.3, 83.2), turned to 90 degrees
- moved C1 129.1 mm to (147.8, 83.2), turned to 90 degrees
- moved C3 125.6 mm to (145.2, 83.2), turned to 90 degrees
- moved SW_BOOT1 124.3 mm to (138.5, 89.0)
- moved C2 122.1 mm to (142.7, 83.2), turned to 90 degrees
- moved L1 118.8 mm to (102.2, 97.5)
- moved C6 117.1 mm to (113.9, 96.4)
- moved C8 117.1 mm to (113.9, 99.4)
- moved C9 117.1 mm to (113.9, 102.4)
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Connections:
- DC_DRIVER2 pad 2: /Motors/DC_1_IN2 -> /Motors/DC_2_IN2
- DC_DRIVER2 pad 3: /Motors/DC_1_IN1 -> /Motors/DC_2_IN1
- DC_DRIVER2 pad 4: Net-(DC_DRIVER1-ILIM) -> Net-(DC_DRIVER2-ILIM)
- DC_DRIVER2 pad 6: Net-(DC_DRIVER1-OUT1) -> Net-(DC_DRIVER2-OUT1)
- DC_DRIVER2 pad 8: Net-(DC_DRIVER1-OUT2) -> Net-(DC_DRIVER2-OUT2)
- DC_DRIVER3 pad 2: /Motors/DC_1_IN2 -> /Motors/DC_3_IN2
- DC_DRIVER3 pad 3: /Motors/DC_1_IN1 -> /Motors/DC_3_IN1
- DC_DRIVER3 pad 4: Net-(DC_DRIVER1-ILIM) -> Net-(DC_DRIVER3-ILIM)
- DC_DRIVER3 pad 6: Net-(DC_DRIVER1-OUT1) -> Net-(DC_DRIVER3-OUT1)
- DC_DRIVER3 pad 8: Net-(DC_DRIVER1-OUT2) -> Net-(DC_DRIVER3-OUT2)
- JP1 pad 2: +5V -> Net-(D1-A)
- Pin_DC_OUT_2 pad 1: Net-(DC_DRIVER1-OUT1) -> Net-(DC_DRIVER2-OUT1)
- Pin_DC_OUT_2 pad 2: Net-(DC_DRIVER1-OUT2) -> Net-(DC_DRIVER2-OUT2)
- Pin_DC_OUT_3 pad 1: Net-(DC_DRIVER1-OUT1) -> Net-(DC_DRIVER3-OUT1)
- Pin_DC_OUT_3 pad 2: Net-(DC_DRIVER1-OUT2) -> Net-(DC_DRIVER3-OUT2)
- R12 pad 1: /Motors/DC_1_IN2 -> /Motors/DC_2_IN2
- R13 pad 1: /Motors/DC_1_IN1 -> /Motors/DC_2_IN1
- R14 pad 2: Net-(DC_DRIVER1-ILIM) -> Net-(DC_DRIVER2-ILIM)
- R15 pad 1: /Motors/DC_1_IN2 -> /Motors/DC_3_IN2
- R16 pad 1: /Motors/DC_1_IN1 -> /Motors/DC_3_IN1
- R17 pad 2: Net-(DC_DRIVER1-ILIM) -> Net-(DC_DRIVER3-ILIM)
- R20 pad 1: GND -> Net-(USB1-A)
- R20 pad 2: Net-(USB_C1-CC1) -> USB
- R21 pad 2: Net-(USB_C1-CC2) -> Net-(USB_C1-CC1)
- R22 pad 1: /Actuators & Utility/STATUS_LED -> GND
- R22 pad 2: Net-(S_ESP1-A) -> Net-(USB_C1-CC2)
- USB_C1 pad A4: +5V -> USB
- USB_C1 pad A9: +5V -> USB
- USB_C1 pad B4: +5V -> USB
- USB_C1 pad B9: +5V -> USB

Commit message: fix: a lot of small things, simplify
Parts:
- removed C18, C19: TBD, Capacitor_SMD:C_0603_1608Metric
- removed LED_strip1: Conn_01x03_Pin, Connector_JST:JST_XH_B3B-XH-A_1x03_P2.50mm_Vertical
- removed R18, R19: TBD, Resistor_SMD:R_0603_1608Metric
- removed Spare_GPIOs1: Conn_01x05_Pin, Connector_PinHeader_1.00mm:PinHeader_1x05_P1.00mm_Vertical
- added C20: 22uF, Capacitor_SMD:C_0201_0603Metric, F.Cu at (156.9, 77.2)
- added C21: 22uF, Capacitor_SMD:C_0201_0603Metric, F.Cu at (156.9, 79.0)
- added C22: 22uF, Capacitor_SMD:C_0201_0603Metric, F.Cu at (156.9, 80.8)
- added C23: 22uF, Capacitor_SMD:C_0201_0603Metric, F.Cu at (156.9, 82.5)
- added R24: 10k, Resistor_SMD:R_0201_0603Metric, F.Cu at (161.4, 82.7)
- added R25: 10k, Resistor_SMD:R_0201_0603Metric, F.Cu at (161.4, 84.5)
- added U1: USBLC6-2P6, Package_TO_SOT_SMD:SOT-666, F.Cu at (162.2, 78.2)
- C10, C11: value 0.1uF -> 1uF
- C2: value 0.22uF -> 22uF
- R20: value 200 -> 1K
- R3: value 20K -> 30K
- moved D1 74.0 mm to (119.5, 108.2), turned to 180 degrees
- moved R23 58.4 mm to (159.6, 126.0)
- moved R22 53.3 mm to (147.1, 74.5)
- moved USB1 43.8 mm to (150.5, 74.5)
- moved D2 43.2 mm to (144.2, 78.2), turned to 180 degrees
- moved C1 4.50 mm to (143.3, 83.0)
- moved C3 4.50 mm to (140.8, 83.0)
- moved R1 4.50 mm to (148.3, 83.0)
- moved C2 4.50 mm to (138.2, 83.0)
- moved R2 4.50 mm to (145.8, 83.0)
- moved L1 2.12 mm to (103.8, 96.0)
- moved SW_ENABLE1 1.46 mm to (151.8, 90.2)
- moved SW_BOOT1 1.35 mm to (138.0, 90.2)
Connections:
- C10 pad 1: +5V -> Net-(D1-K)
- D1 pad 1: +5V -> Net-(D1-K)
- D1 pad 2: Net-(D1-A) -> +5V
- D2 pad 1: +5V -> Net-(D1-K)
- ESP32-S3-WROOM1 pad 16: /Actuators & Utility/SERVO_3 -> Net-(ESP32-S3-WROOM1-IO46)
- ESP32-S3-WROOM1 pad 18: /Actuators & Utility/IO14 -> unconnected-(ESP32-S3-WROOM1-IO10-Pad18)
- ESP32-S3-WROOM1 pad 19: /Actuators & Utility/IO13 -> unconnected-(ESP32-S3-WROOM1-IO11-Pad19)
- ESP32-S3-WROOM1 pad 20: /Actuators & Utility/IO12 -> unconnected-(ESP32-S3-WROOM1-IO12-Pad20)
- ESP32-S3-WROOM1 pad 21: /Actuators & Utility/IO11 -> unconnected-(ESP32-S3-WROOM1-IO13-Pad21)
- ESP32-S3-WROOM1 pad 22: /Actuators & Utility/IO10 -> /Actuators & Utility/SERVO_3
- ESP32-S3-WROOM1 pad 26: /Actuators & Utility/SERVO_4 -> Net-(ESP32-S3-WROOM1-IO45)
- ESP32-S3-WROOM1 pad 8: /Actuators & Utility/LED_STRIP -> /Actuators & Utility/SERVO_4
- JP1 pad 2: Net-(D1-A) -> +5V
- LDO1 pad 1: +5V -> Net-(D1-K)
- LDO1 pad 3: +5V -> Net-(D1-K)
- USB_C1 pad A6: Net-(R19-Pad2) -> /External IO/USB_D+
- USB_C1 pad A7: Net-(R18-Pad2) -> /External IO/USB_D-
- USB_C1 pad B6: Net-(R19-Pad2) -> /External IO/USB_D+
- USB_C1 pad B7: Net-(R18-Pad2) -> /External IO/USB_D-

Commit message: better layout
Parts:
- removed the SERVO_4 at (164.0, 104.8)
- added SERVO_1: Conn_01x03_Pin, Connector_JST:JST_XH_B3B-XH-A_1x03_P2.50mm_Vertical, F.Cu at (91.0, 67.5)
- C20, C21, C22, C23: footprint Capacitor_SMD:C_0201_0603Metric -> Capacitor_SMD:C_0603_1608Metric
- moved SERVO_3 78.7 mm to (91.0, 95.5), turned to 0 degrees
- moved C23 73.0 mm to (92.0, 116.0)
- moved I2C1 69.8 mm to (162.5, 99.0), turned to 0 degrees
- moved C22 68.1 mm to (92.2, 102.0)
- moved C21 65.5 mm to (92.0, 88.0)
- moved C20 65.0 mm to (92.0, 74.0)
- moved SERVO_4 29.5 mm to (91.0, 109.5), turned to 0 degrees
- moved SPI1 23.0 mm to (159.0, 88.0), turned to 0 degrees
- moved R21 16.4 mm to (161.0, 66.8)
- moved R22 16.4 mm to (159.1, 63.3)
- moved USB1 16.4 mm to (162.6, 63.3)
- moved D2 16.4 mm to (156.2, 67.1)
- moved R20 16.4 mm to (163.5, 66.8)
- moved SW_BOOT1 15.0 mm to (123.0, 90.2)
- moved SW_ENABLE1 15.0 mm to (136.8, 90.2)
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- renumbered SERVO_1 to SERVO_4
Connections:
- SERVO_4 pad 3: /Actuators & Utility/SERVO_1 -> /Actuators & Utility/SERVO_4

Commit message: Routing V1 done
Parts:
- added C18: 1uF, Capacitor_SMD:C_0603_1608Metric, F.Cu at (96.1, 88.4)
- added J1: Conn_01x04_Pin, Connector_PinHeader_1.00mm:PinHeader_1x04_P1.00mm_Vertical, F.Cu at (146.6, 83.8)
- C20, C21, C22, C23: footprint Capacitor_SMD:C_0603_1608Metric -> Capacitor_SMD:C_0805_2012Metric
- R2: footprint Resistor_SMD:R_0603_1608Metric -> Resistor_SMD:R_0805_2012Metric
- R20: footprint Resistor_SMD:R_0603_1608Metric_Pad0.98x0.95mm_HandSolder -> PCM_SparkFun-Resistor:R_0603_1608Metric
- R24: footprint Resistor_SMD:R_0201_0603Metric -> PCM_SparkFun-Resistor:R_0603_1608Metric
- R25: footprint Resistor_SMD:R_0201_0603Metric -> Resistor_SMD:R_0603_1608Metric
- moved H4 122.5 mm to (179.2, 133.5)
- moved H2 115.0 mm to (179.2, 68.1)
- moved USB_C1 86.4 mm to (86.8, 81.4), turned to -90 degrees
- moved I2C1 78.4 mm to (90.7, 67.5)
- moved USB1 77.0 mm to (90.1, 89.1)
- moved C22 73.0 mm to (165.2, 99.9), turned to 180 degrees
- moved C23 73.0 mm to (164.9, 113.9), turned to 180 degrees
- moved SERVO_3 73.0 mm to (163.9, 93.4)
- moved SERVO_4 73.0 mm to (163.9, 107.4)
- moved R20 72.7 mm to (94.0, 88.4), turned to 90 degrees
- moved U1 69.1 mm to (93.3, 81.3)
- moved R21 67.6 mm to (94.0, 75.6)
- moved R22 63.5 mm to (96.8, 75.6), turned to -90 degrees
- moved H3 62.0 mm to (80.5, 133.5)
- moved D2 58.4 mm to (100.3, 83.8)
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- renumbered Pin_DC_OUT_1 to DC_OUT_1, Pin_DC_OUT_2 to DC_OUT_2, Pin_DC_OUT_3 to DC_OUT_3
Connections:
- ESP32-S3-WROOM1 pad 18: unconnected-(ESP32-S3-WROOM1-IO10-Pad18) -> /Actuators & Utility/GPIO4
- ESP32-S3-WROOM1 pad 19: unconnected-(ESP32-S3-WROOM1-IO11-Pad19) -> /Actuators & Utility/GPIO3
- ESP32-S3-WROOM1 pad 20: unconnected-(ESP32-S3-WROOM1-IO12-Pad20) -> /Actuators & Utility/GPIO2
- ESP32-S3-WROOM1 pad 21: unconnected-(ESP32-S3-WROOM1-IO13-Pad21) -> /Actuators & Utility/GPIO1
- ESP32-S3-WROOM1 pad 24: /Actuators & Utility/SERVO_2 -> /Actuators & Utility/SERVO_1
- ESP32-S3-WROOM1 pad 25: /Actuators & Utility/SERVO_1 -> /Actuators & Utility/SERVO_2
- SPI1 pad 2: /External IO/MOSI -> /External IO/CS
- SPI1 pad 3: /External IO/MISO -> /External IO/Handshake
- SPI1 pad 4: /External IO/CS -> /External IO/MISO
- SPI1 pad 5: /External IO/Handshake -> /External IO/MOSI
- U1 pad 1: /External IO/USB_D+ -> Net-(U1-I/O1-Pad1)
- U1 pad 3: /External IO/USB_D- -> Net-(U1-I/O2-Pad3)
- U1 pad 4: /External IO/USB_D- -> /External IO/USB_D+
- U1 pad 6: /External IO/USB_D+ -> /External IO/USB_D-
- UART1 pad 2: /External IO/RXD0 -> /External IO/TXD0
- UART1 pad 3: /External IO/TXD0 -> /External IO/RXD0
- USB_C1 pad A6: /External IO/USB_D+ -> Net-(U1-I/O2-Pad3)
- USB_C1 pad A7: /External IO/USB_D- -> Net-(U1-I/O1-Pad1)
- USB_C1 pad B6: /External IO/USB_D+ -> Net-(U1-I/O2-Pad3)
- USB_C1 pad B7: /External IO/USB_D- -> Net-(U1-I/O1-Pad1)
Routing:
- net BATT: track 0.00 -> 304.9 mm, vias 0 -> 7
- net +3.3V: track 0.00 -> 181.9 mm, vias 0 -> 3
- net +5V: track 0.00 -> 177.3 mm, vias 0 -> 2
- net /Actuators & Utility/STATUS_LED: track 0.00 -> 118.1 mm, vias 0 -> 2
- net /Actuators & Utility/SERVO_4: track 0.00 -> 69.3 mm, vias 0 -> 1
- net GND: track 0.00 -> 67.0 mm, vias 0 -> 212
- net /Actuators & Utility/SERVO_2: track 0.00 -> 60.9 mm, vias 0 -> 4
- net /Motors/DC_3_IN1: track 0.00 -> 60.8 mm, vias 0 -> 2
- net /Motors/DC_2_IN1: track 0.00 -> 60.5 mm, vias 0 -> 2
- net /Motors/DC_2_IN2: track 0.00 -> 59.5 mm, vias 0 -> 2
- net /Motors/DC_1_IN1: track 0.00 -> 55.9 mm, vias 0 -> 2
- net /Motors/DC_1_IN2: track 0.00 -> 54.7 mm, vias 0 -> 2
- net /Actuators & Utility/SERVO_1: track 0.00 -> 54.4 mm, vias 0 -> 4
- net /Motors/DC_3_IN2: track 0.00 -> 53.8 mm, vias 0 -> 2
- net /Actuators & Utility/SERVO_3: track 0.00 -> 48.1 mm, vias 0 -> 1
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- added copper zone on In1.Cu, net (none)
- added copper zone on B.Cu, net GND
- added copper zone on F.Cu, net GND
- added copper zone on In2.Cu, net GND
Other:
- board outline added: 109.8 x 79.6 mm

Commit message: cleanup
Parts:
- I2C1: moved to B.Cu
- moved I2C1 7.73 mm to (98.4, 67.6), turned to 180 degrees
- moved C18 7.55 mm to (88.5, 88.2)
- moved D2 7.55 mm to (92.7, 83.6)
- moved R21 7.55 mm to (86.5, 75.4)
- moved R22 7.55 mm to (89.2, 75.4)
- moved USB1 7.55 mm to (82.5, 88.9)
- moved USB_C1 7.55 mm to (79.2, 81.2)
- moved R20 7.55 mm to (86.5, 88.2)
- moved U1 7.55 mm to (85.8, 81.1)
Routing:
- net /External IO/SCL: track 42.4 -> 34.7 mm
- net /External IO/USB_D-: track 24.2 -> 31.8 mm
- net /External IO/USB_D+: track 24.1 -> 31.8 mm
- net Net-(D1-K): track 20.3 -> 27.9 mm
- net /External IO/SDA: track 37.4 -> 34.6 mm
- net +3.3V: track 181.9 -> 183.0 mm
- net GND: track 67.0 -> 67.2 mm, vias 212 -> 228

Commit message: text
Parts:
- added REF**: KiCad-Logo2_6mm_SilkScreen, Symbol:KiCad-Logo2_6mm_SilkScreen, B.Cu at (166.3, 128.6)
- UART1: footprint Connector_JST:JST_XH_B4B-XH-A_1x04_P2.50mm_Vertical -> Connector_PinHeader_1.00mm:PinHeader_1x04_P1.00mm_Vertical
- moved UART1 3.99 mm to (166.2, 66.7)
- moved TP4 0.18 mm to (160.8, 134.6)
Connections:
- net /Actuators & Utility/GPIO1 renamed /Actuators & Utility/GPIO13
- net /Actuators & Utility/GPIO2 renamed /Actuators & Utility/GPIO12
- net /Actuators & Utility/GPIO3 renamed /Actuators & Utility/GPIO11
- net /Actuators & Utility/GPIO4 renamed /Actuators & Utility/GPIO10
Routing:
- net +3.3V: track 183.0 -> 179.7 mm
- net /External IO/RXD0: track 34.6 -> 31.5 mm
- net GND: vias 228 -> 227
Other:
- board text added: "3.3V"
- board text added: "5V"
- board text added: "BATT"
- board text added: "BATTERY"
- board text added: "BAU"
- board text added: "BOOT"
- board text added: "BUCK 5V"
- board text added: "CLK"
- board text added: "CS"
- board text added: "Carte de contrôle V1 PAMIs CDFR 2027"
- board text added: "DC 1 OUTPUT"
- board text added: "DC 2 OUTPUT"
- board text added: "DC 3 OUTPUT"
- board text added: "DC DRIVER 1"
- board text added: "DC DRIVER 2"
- board text added: "DC DRIVER 3"
- board text added: "ENABLE"
- board text added: "ESP"
- board text added: "GND"
- board text added: "GPIO10"
- board text added: "GPIO11"
- board text added: "GPIO12"
- board text added: "GPIO13"
- board text added: "HS"
- board text added: "I2C OTOS"
- board text added: "LDO 3.3V"
- board text added: "MISO"
- board text added: "MOSI"
- board text added: "OUT1"
- board text added: "OUT2"
- board text added: "PIERSON Robin"
- board text added: "RX"
- board text added: "SCL"
- board text added: "SDA"
- board text added: "SIGNAL"
- board text added: "SPARE GPIOs"
- board text added: "SPI"
- board text added: "STATUS LEDs"
- board text added: "TX"
- board text added: "UART"
- board text added: "USB"
