File: ControlBoard/CDFR2027-PAMIs-ELEC-control.kicad_pcb (KiCad board)
At the start: 4 copper layers, 80.4 x 79.8 mm, 92 parts, among them J1 Conn_01x04_Pin, Q1 PMOS, U1 USBLC6-2P6

Commit message: (fix): kicad logo too low
Parts:
- moved REF** 0.78 mm to (124.5, 107.8)
Changed lines of the file:
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@@
 	(footprint "Symbol:KiCad-Logo2_6mm_SilkScreen"
 		(layer "B.Cu")
-		(at 124.543272 108.592526 180)
+		(at 124.5 107.81 180)
 		(descr "KiCad Logo")
 		(tags "Logo KiCad")

Commit message: (prod): final adjustements and final bom for production
Parts:
- removed J1: Conn_01x04_Pin, Connector_PinHeader_1.00mm:PinHeader_1x04_P1.00mm_Vertical
- UART1: footprint Connector_PinHeader_1.00mm:PinHeader_1x04_P1.00mm_Vertical -> Connector_PinHeader_2.54mm:PinHeader_1x04_P2.54mm_Vertical
- moved UART1 0.59 mm to (139.4, 84.3)
Connections:
- ESP32-S3-WROOM1 pad 18: /Actuators & Utility/GPIO10 -> unconnected-(ESP32-S3-WROOM1-IO10-Pad18)
- ESP32-S3-WROOM1 pad 19: /Actuators & Utility/GPIO11 -> unconnected-(ESP32-S3-WROOM1-IO11-Pad19)
- ESP32-S3-WROOM1 pad 20: /Actuators & Utility/GPIO12 -> unconnected-(ESP32-S3-WROOM1-IO12-Pad20)
- ESP32-S3-WROOM1 pad 21: /Actuators & Utility/GPIO13 -> unconnected-(ESP32-S3-WROOM1-IO13-Pad21)
- Q1 pad 4: Net-(Q1-D) -> (no net)
Routing:
- net +3.3V: track 109.8 -> 114.7 mm
- net /External IO/RXD0: track 9.28 -> 13.9 mm
- net /Actuators & Utility/GPIO10: track 3.11 -> 0.00 mm
- net /Actuators & Utility/GPIO11: track 3.00 -> 0.00 mm
- net /Actuators & Utility/GPIO13: track 2.93 -> 0.00 mm
- net /Actuators & Utility/GPIO12: track 2.89 -> 0.00 mm
- net /External IO/TXD0: track 8.16 -> 10.5 mm
- net BATT: track 245.7 -> 247.6 mm
- net GND: vias 264 -> 263
Other:
- board text removed: "SPARE GPIO"
