File: ControlBoard/actuators.kicad_sch (KiCad schematic)
At the start: 9 parts, among them J1 Conn_01x03_Pin, J3 Conn_01x03_Pin, J4 Conn_01x03_Pin, J5 Conn_01x03_Pin, J6 Conn_01x03_Pin, J8 Conn_01x05_Pin

Commit message: WIP: placement
Parts:
- LED_strip1: renamed from J1; footprint (none) -> Connector_JST:JST_XH_B3B-XH-A_1x03_P2.50mm_Vertical
- SERVO_1: renamed from J3; footprint (none) -> Connector_JST:JST_XH_B3B-XH-A_1x03_P2.50mm_Vertical
- SERVO_2: renamed from J4; footprint (none) -> Connector_JST:JST_XH_B3B-XH-A_1x03_P2.50mm_Vertical
- SERVO_3: renamed from J5; footprint (none) -> Connector_JST:JST_XH_B3B-XH-A_1x03_P2.50mm_Vertical
- SERVO_4: renamed from J6; footprint (none) -> Connector_JST:JST_XH_B3B-XH-A_1x03_P2.50mm_Vertical
- Spare_GPIOs1: renamed from J8; footprint (none) -> Connector_PinHeader_1.00mm:PinHeader_1x05_P1.00mm_Vertical
- renumbered R13 to R22, TP5 to TP4
Connections:
- net SERVO_A renamed SERVO_1
- net SERVO_B renamed SERVO_2
- net SERVO_C renamed SERVO_3
- net SERVO_D renamed SERVO_4
Other:
- moved on the sheet: LED_strip1, R22, SERVO_1, SERVO_2, SERVO_3, SERVO_4, S_ESP1, Spare_GPIOs1, TP4

Commit message: Feat: multiplex power over usb + add gitignore
Parts:
- renumbered R22 to R23
Changed lines of the file:
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@@
 		(dnp no)
 		(fields_autoplaced yes)
-		(property "Reference" "#PWR048"
+		(property "Reference" "#PWR050"
 			(at 129.54 113.03 0)
 			(hide yes)
@@
 			(project "CDFR2027-PAMIs-ELEC-control"
 				(path "/e464473e-1f11-4961-9962-67415e223b13/69c65a6e-fa15-49ab-aaed-4f63cbee0221"
-					(reference "#PWR048")
+					(reference "#PWR050")
 					(unit 1)
 				)
@@
 		(dnp no)
 		(fields_autoplaced yes)
-		(property "Reference" "#PWR044"
+		(property "Reference" "#PWR046"
 			(at 129.54 88.9 0)
 			(hide yes)
@@
 			(project "CDFR2027-PAMIs-ELEC-control"
 				(path "/e464473e-1f11-4961-9962-67415e223b13/69c65a6e-fa15-49ab-aaed-4f63cbee0221"
-					(reference "#PWR044")
+					(reference "#PWR046")
 					(unit 1)
 				)
@@
 		(dnp no)
 		(fields_autoplaced yes)
-		(property "Reference" "#PWR041"
+		(property "Reference" "#PWR043"
 			(at 139.7 73.66 0)
 			(hide yes)
@@
 			(project "CDFR2027-PAMIs-ELEC-control"
 				(path "/e464473e-1f11-4961-9962-67415e223b13/69c65a6e-fa15-49ab-aaed-4f63cbee0221"
-					(reference "#PWR041")
+					(reference "#PWR043")
 					(unit 1)
 				)
@@
 		(dnp no)
 		(fields_autoplaced yes)
-		(property "Reference" "#PWR050"
+		(property "Reference" "#PWR052"
 			(at 173.99 76.2 0)
 			(hide yes)
@@
 			(project "CDFR2027-PAMIs-ELEC-control"
 				(path "/e464473e-1f11-4961-9962-67415e223b13/69c65a6e-fa15-49ab-aaed-4f63cbee0221"
-					(reference "#PWR050")
+					(reference "#PWR052")
 					(unit 1)
 				)
@@
 		(dnp no)
 		(fields_autoplaced yes)
-		(property "Reference" "#PWR049"
+		(property "Reference" "#PWR051"
 			(at 184.15 73.66 0)
 			(hide yes)
@@
 			(project "CDFR2027-PAMIs-ELEC-control"
 				(path "/e464473e-1f11-4961-9962-67415e223b13/69c65a6e-fa15-49ab-aaed-4f63cbee0221"
-					(reference "#PWR049")
+					(reference "#PWR051")
 					(unit 1)
 				)
@@
 		(dnp no)
 		(fields_autoplaced yes)
-		(property "Reference" "#PWR047"
+		(property "Reference" "#PWR049"
 			(at 139.7 110.49 0)
 			(hide yes)
@@
 			(project "CDFR2027-PAMIs-ELEC-control"
 				(path "/e464473e-1f11-4961-9962-67415e223b13/69c65a6e-fa15-49ab-aaed-4f63cbee0221"
-					(reference "#PWR047")
+					(reference "#PWR049")
 					(unit 1)
 				)
@@
 		(dnp no)
 		(fields_autoplaced yes)
-		(property "Reference" "R22"
+		(property "Reference" "R23"
 			(at 105.41 97.7899 0)
 			(show_name no)
@@
 			(project "CDFR2027-PAMIs-ELEC-control"
 				(path "/e464473e-1f11-4961-9962-67415e223b13/69c65a6e-fa15-49ab-aaed-4f63cbee0221"
-					(reference "R22")
+					(reference "R23")
 					(unit 1)
 				)
@@
 		(dnp no)
 		(fields_autoplaced yes)
-		(property "Reference" "#PWR045"
+		(property "Reference" "#PWR047"
 			(at 139.7 99.06 0)
 			(hide yes)
@@
 			(project "CDFR2027-PAMIs-ELEC-control"
 				(path "/e464473e-1f11-4961-9962-67415e223b13/69c65a6e-fa15-49ab-aaed-4f63cbee0221"
-					(reference "#PWR045")
+					(reference "#PWR047")
 					(unit 1)
 				)
@@
 		(dnp no)
 		(fields_autoplaced yes)
-		(property "Reference" "#PWR046"
+		(property "Reference" "#PWR048"
 			(at 129.54 101.6 0)
 			(hide yes)
@@
 			(project "CDFR2027-PAMIs-ELEC-control"
 				(path "/e464473e-1f11-4961-9962-67415e223b13/69c65a6e-fa15-49ab-aaed-4f63cbee0221"
-					(reference "#PWR046")
+					(reference "#PWR048")
 					(unit 1)
 				)
@@
 		(dnp no)
 		(fields_autoplaced yes)
-		(property "Reference" "#PWR042"
+		(property "Reference" "#PWR044"
 			(at 129.54 76.2 0)
 			(hide yes)
@@
 			(project "CDFR2027-PAMIs-ELEC-control"
 				(path "/e464473e-1f11-4961-9962-67415e223b13/69c65a6e-fa15-49ab-aaed-4f63cbee0221"
-					(reference "#PWR042")
+					(reference "#PWR044")
 					(unit 1)
 				)
@@
 		(dnp no)
 		(fields_autoplaced yes)
-		(property "Reference" "#PWR043"
+		(property "Reference" "#PWR045"
 			(at 139.7 86.36 0)
 			(hide yes)
@@
 			(project "CDFR2027-PAMIs-ELEC-control"
 				(path "/e464473e-1f11-4961-9962-67415e223b13/69c65a6e-fa15-49ab-aaed-4f63cbee0221"
-					(reference "#PWR043")
+					(reference "#PWR045")
 					(unit 1)
 				)
@@
 		(dnp no)
 		(fields_autoplaced yes)
-		(property "Reference" "#PWR040"
+		(property "Reference" "#PWR042"
 			(at 102.87 119.38 0)
 			(hide yes)
@@
 			(project "CDFR2027-PAMIs-ELEC-control"
 				(path "/e464473e-1f11-4961-9962-67415e223b13/69c65a6e-fa15-49ab-aaed-4f63cbee0221"
-					(reference "#PWR040")
-					(unit 1)
-				)
+					(reference "#PWR042")
+					(unit 1)
+				)

Commit message: fix: a lot of small things, simplify
Parts:
- removed LED_strip1: Conn_01x03_Pin, Connector_JST:JST_XH_B3B-XH-A_1x03_P2.50mm_Vertical, symbol Connector:Conn_01x03_Pin
- removed Spare_GPIOs1: Conn_01x05_Pin, Connector_PinHeader_1.00mm:PinHeader_1x05_P1.00mm_Vertical, symbol Connector:Conn_01x05_Pin
- added C20, C21, C22, C23: 22uF, Capacitor_SMD:C_0201_0603Metric, symbol Device:C
Connections:
- net +5V: now also C20.1, C21.1, C22.1, C23.1
- net GND: now also C20.2, C21.2, C22.2, C23.2
Other:
- moved on the sheet: R23, SERVO_1, S_ESP1, TP4

Commit message: better layout
Parts:
- C20, C21, C22, C23: footprint Capacitor_SMD:C_0201_0603Metric -> Capacitor_SMD:C_0603_1608Metric
Changed lines of the file:
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@@
 			)
 		)
-		(property "Footprint" "Capacitor_SMD:C_0201_0603Metric"
+		(property "Footprint" "Capacitor_SMD:C_0603_1608Metric"
 			(at 143.2052 90.17 0)
 			(hide yes)
@@
 			)
 		)
-		(property "Footprint" "Capacitor_SMD:C_0201_0603Metric"
+		(property "Footprint" "Capacitor_SMD:C_0603_1608Metric"
 			(at 143.2052 113.03 0)
 			(hide yes)
@@
 			)
 		)
-		(property "Footprint" "Capacitor_SMD:C_0201_0603Metric"
+		(property "Footprint" "Capacitor_SMD:C_0603_1608Metric"
 			(at 143.2052 66.04 0)
 			(hide yes)
@@
 			)
 		)
-		(property "Footprint" "Capacitor_SMD:C_0201_0603Metric"
+		(property "Footprint" "Capacitor_SMD:C_0603_1608Metric"
 			(at 143.2052 135.89 0)
 			(hide yes)

Commit message: Routing V1 done
Parts:
- added J1: Conn_01x04_Pin, Connector_PinHeader_1.00mm:PinHeader_1x04_P1.00mm_Vertical, symbol Connector:Conn_01x04_Pin
- C20, C21, C22, C23: footprint Capacitor_SMD:C_0603_1608Metric -> Capacitor_SMD:C_0805_2012Metric
Connections:
- new net GPIO1: J1.4 (Pin_4)
- new net GPIO2: J1.3 (Pin_3)
- new net GPIO3: J1.2 (Pin_2)
- new net GPIO4: J1.1 (Pin_1)

Commit message: text
Connections:
- net GPIO1 renamed GPIO13
- net GPIO2 renamed GPIO12
- net GPIO3 renamed GPIO11
- net GPIO4 renamed GPIO10
Changed lines of the file:
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@@
 	(text_box "Spare GPIOs\n"
 		(exclude_from_sim no)
-		(at 93.98 92.71 0)
-		(size 31.75 15.24)
+		(at 91.44 92.71 0)
+		(size 34.29 15.24)
 		(margins 0.9525 0.9525 0.9525 0.9525)
 		(stroke
@@
 		)
 	)
-	(hierarchical_label "GPIO1"
+	(hierarchical_label "GPIO13"
 		(shape input)
 		(at 102.87 97.79 180)
@@
 		)
 	)
-	(hierarchical_label "GPIO3"
+	(hierarchical_label "GPIO11"
 		(shape input)
 		(at 102.87 102.87 180)
@@
 		)
 	)
-	(hierarchical_label "GPIO4"
+	(hierarchical_label "GPIO10"
 		(shape input)
 		(at 102.87 105.41 180)
@@
 		)
 	)
-	(hierarchical_label "GPIO2"
+	(hierarchical_label "GPIO12"
 		(shape input)
 		(at 102.87 100.33 180)

Commit message: (feat): bom
Parts:
- J1: LCSC (none) -> C52016392
- SERVO_1, SERVO_2, SERVO_3, SERVO_4: LCSC (none) -> C144394
Changed lines of the file:
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@@
+			)
+		)
+		(property "LCSC" "C144394"
+			(at 156.21 80.01 0)
+			(hide yes)
+			(show_name no)
+			(do_not_autoplace no)
+			(effects
+				(font
+					(size 1.27 1.27)
+				)
 			)
 		)
@@
 			)
 		)
+		(property "LCSC" "C52016392"
+			(at 107.95 102.87 0)
+			(hide yes)
+			(show_name no)
+			(do_not_autoplace no)
+			(effects
+				(font
+					(size 1.27 1.27)
+				)
+			)
+		)
 		(pin "1"
 		)
@@
 			)
 		)
+		(property "LCSC" "C144394"
+			(at 156.21 125.73 0)
+			(hide yes)
+			(show_name no)
+			(do_not_autoplace no)
+			(effects
+				(font
+					(size 1.27 1.27)
+				)
+			)
+		)
 		(pin "2"
 		)
@@
 			)
 		)
+		(property "LCSC" "C144394"
+			(at 156.21 102.87 0)
+			(hide yes)
+			(show_name no)
+			(do_not_autoplace no)
+			(effects
+				(font
+					(size 1.27 1.27)
+				)
+			)
+		)
 		(pin "2"
 		)
@@
 			(at 156.21 55.88 0)
 			(hide yes)
+			(show_name no)
+			(do_not_autoplace no)
+			(effects
+				(font
+					(size 1.27 1.27)
+				)
+			)
+		)
+		(property "LCSC" "C144394"
+			(at 156.21 55.88 0)
+			(hide yes)

Commit message: Updates to schematic by Ludo <3
Changed lines of the file:
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@@
 		(property "Value" "GND"
 			(at 142.24 74.422 0)
+			(hide yes)
 			(show_name no)
 			(do_not_autoplace no)
@@
 		(property "Value" "GND"
 			(at 142.24 121.412 0)
+			(hide yes)
 			(show_name no)
 			(do_not_autoplace no)
@@
 		(property "Value" "GND"
 			(at 142.24 98.552 0)
+			(hide yes)
 			(show_name no)
 			(do_not_autoplace no)
@@
 		(property "Value" "GND"
 			(at 142.24 144.272 0)
-			(show_name no)
-			(do_not_autoplace no)
+			(hide yes)
+			(show_name no)
+			(do_not_autoplace no)
