File: ControlBoard/io.kicad_sch (KiCad schematic)
At the start: 10 parts, among them J2 Conn_01x04_Pin, J7 USB_C_Receptacle_USB2.0_14P

Commit message: WIP: placement
Parts:
- C18: renamed from C21; footprint Package_SO:SOIC-8_3.9x4.9mm_P1.27mm -> Capacitor_SMD:C_0603_1608Metric
- C19: renamed from C22; footprint Package_SO:SOIC-8_3.9x4.9mm_P1.27mm -> Capacitor_SMD:C_0603_1608Metric
- I2C1: footprint (none) -> Connector_JST:JST_XH_B4B-XH-A_1x04_P2.50mm_Vertical
- R18: renamed from R23; footprint Package_DIP:DIP-8_W7.62mm -> Resistor_SMD:R_0603_1608Metric
- R19: renamed from R24; footprint Package_DIP:DIP-8_W7.62mm -> Resistor_SMD:R_0603_1608Metric
- R20: renamed from R25; footprint Package_DIP:DIP-8_W7.62mm -> Resistor_SMD:R_0603_1608Metric
- R21: renamed from R26; footprint Package_DIP:DIP-8_W7.62mm -> Resistor_SMD:R_0603_1608Metric
- SPI1: footprint (none) -> Connector_JST:JST_XH_B7B-XH-A_1x07_P2.50mm_Vertical
- UART1: renamed from J2; footprint (none) -> Connector_JST:JST_XH_B4B-XH-A_1x04_P2.50mm_Vertical
- USB_C1: renamed from J7; footprint Package_DFN_QFN:WDFN-10-1EP_3x3mm_P0.5mm_EP1.8x2.5mm -> Connector_USB:USB_C_Receptacle_G-Switch_GT-USB-7051x

Commit message: Feat: multiplex power over usb + add gitignore
Parts:
- added R20: 200, Resistor_SMD:R_0603_1608Metric_Pad0.98x0.95mm_HandSolder, symbol Device:R
- added USB1: LED, Diode_SMD:D_0603_1608Metric, symbol Device:LED
- USB_C1: footprint Connector_USB:USB_C_Receptacle_G-Switch_GT-USB-7051x -> Connector_USB:USB_C_Receptacle_GCT_USB4105-xx-A_16P_TopMnt_Horizontal
- renumbered R20 to R21, R21 to R22
Connections:
- net GND: now also USB1.1 (K)
- net +5V renamed USB
- net USB: now also R20.2
- new net: R20.1, USB1.2 (A)
Other:
- moved on the sheet: C18, C19, R18, R19, R21, R22, USB_C1

Commit message: fix: a lot of small things, simplify
Parts:
- removed C18, C19: TBD, Capacitor_SMD:C_0603_1608Metric, symbol Device:C
- removed R18, R19: TBD, Resistor_SMD:R_0603_1608Metric, symbol Device:R
- added U1: USBLC6-2P6, Package_TO_SOT_SMD:SOT-666, symbol Power_Protection:USBLC6-2P6
- R20: value 200 -> 1K
Connections:
- net GND: now also U1.2 (GND)
- net USB: now also U1.5 (VBUS)
- net USB_D+: now also USB_C1.A6 (D+), USB_C1.B6 (D+), U1.1 (I/O1), U1.6 (I/O1)
- net USB_D-: now also USB_C1.A7 (D-), USB_C1.B7 (D-), U1.3 (I/O2), U1.4 (I/O2)

Commit message: Routing V1 done
Parts:
- added C18: 1uF, Capacitor_SMD:C_0603_1608Metric, symbol Device:C
- R20: footprint Resistor_SMD:R_0603_1608Metric_Pad0.98x0.95mm_HandSolder -> PCM_SparkFun-Resistor:R_0603_1608Metric
Connections:
- net CS: now also SPI1.2 (Pin_2); no longer SPI1.4 (Pin_4)
- net GND: now also C18.1
- net Handshake: now also SPI1.3 (Pin_3); no longer SPI1.5 (Pin_5)
- net MISO: now also SPI1.4 (Pin_4); no longer SPI1.3 (Pin_3)
- net MOSI: now also SPI1.5 (Pin_5); no longer SPI1.2 (Pin_2)
- net RXD0: now also UART1.3 (Pin_3); no longer UART1.2 (Pin_2)
- net TXD0: now also UART1.2 (Pin_2); no longer UART1.3 (Pin_3)
- net USB: now also C18.2
- net USB_D+: now also U1.4 (I/O2); no longer U1.1 (I/O1), U1.6 (I/O1), USB_C1.A6 (D+), USB_C1.B6 (D+)
- net USB_D-: now also U1.6 (I/O1); no longer U1.3 (I/O2), U1.4 (I/O2), USB_C1.A7 (D-), USB_C1.B7 (D-)
- new net: U1.3 (I/O2), USB_C1.A6 (D+), USB_C1.B6 (D+)
- new net: U1.1 (I/O1), USB_C1.A7 (D-), USB_C1.B7 (D-)
Other:
- moved on the sheet: R20, U1, USB1

Commit message: text
Parts:
- UART1: footprint Connector_JST:JST_XH_B4B-XH-A_1x04_P2.50mm_Vertical -> Connector_PinHeader_1.00mm:PinHeader_1x04_P1.00mm_Vertical
Other:
- moved on the sheet: C18, R20, R21, R22, U1, USB1, USB_C1

Commit message: (feat): bom
Parts:
- C18: LCSC (none) -> C1592
- I2C1: LCSC (none) -> C144395
- R20: LCSC (none) -> C22548
- R21, R22: LCSC (none) -> C2907044
- SPI1: LCSC (none) -> C144398
- U1: LCSC (none) -> C15999
- UART1: LCSC (none) -> C52016392
- USB1: LCSC (none) -> C22371297
- USB_C1: LCSC (none) -> C3151746
Changed lines of the file:
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@@
+			)
+		)
+		(property "LCSC" "C144395"
+			(at 180.34 68.58 0)
+			(hide yes)
+			(show_name no)
+			(do_not_autoplace no)
+			(effects
+				(font
+					(size 1.27 1.27)
+				)
 			)
 		)
@@
 			)
 		)
+		(property "LCSC" "C144398"
+			(at 185.42 113.03 0)
+			(hide yes)
+			(show_name no)
+			(do_not_autoplace no)
+			(effects
+				(font
+					(size 1.27 1.27)
+				)
+			)
+		)
 		(pin "1"
 		)
@@
 		)
 		(property "Description" "Resistor"
+			(at 93.98 71.12 0)
+			(hide yes)
+			(show_name no)
+			(do_not_autoplace no)
+			(effects
+				(font
+					(size 1.27 1.27)
+				)
+			)
+		)
+		(property "LCSC" "C22548"
 			(at 93.98 71.12 0)
 			(hide yes)
@@
 			)
 		)
+		(property "LCSC" "C52016392"
+			(at 179.07 88.9 0)
+			(hide yes)
+			(show_name no)
+			(do_not_autoplace no)
+			(effects
+				(font
+					(size 1.27 1.27)
+				)
+			)
+		)
 		(pin "3"
 		)
@@
 		(property "Description" "Resistor"
 			(at 118.11 82.55 0)
+			(hide yes)
+			(show_name no)
+			(do_not_autoplace no)
+			(effects
+				(font
+					(size 1.27 1.27)
+				)
+			)
+		)
+		(property "LCSC" "C2907044"
+			(at 118.11 82.55 90)
 			(hide yes)
 			(show_name no)
@@
 			)
 		)
+		(property "LCSC" "C1592"
+			(at 106.68 71.12 0)
+			(hide yes)
+			(show_name no)
+			(do_not_autoplace no)
+			(effects
+				(font
+					(size 1.27 1.27)
+				)
+			)
+		)
 		(pin "1"
 		)
@@
 			)
 		)
+		(property "LCSC" "C3151746"
+			(at 137.16 92.71 0)
+			(hide yes)
+			(show_name no)
+			(do_not_autoplace no)
+			(effects
+				(font
+					(size 1.27 1.27)
+				)
+			)
+		)
 		(pin "A9"
 		)
@@
 			)
 		)
+		(property "LCSC" "C15999"
+			(at 93.98 90.17 0)
+			(hide yes)
+			(show_name no)
+			(do_not_autoplace no)
+			(effects
+				(font
+					(size 1.27 1.27)
+				)
+			)
+		)
 		(pin "1"
 		)
@@
 			)
 		)
+		(property "LCSC" "C22371297"
+			(at 93.98 63.5 0)
+			(hide yes)
+			(show_name no)
+			(do_not_autoplace no)
+			(effects
+				(font
+					(size 1.27 1.27)
+				)
+			)
+		)
 		(pin "1"
 		)
@@
 			(hide yes)
 			(show_name no)
+			(do_not_autoplace no)
+			(effects
+				(font
+					(size 1.27 1.27)
+				)
+			)
+		)
+		(property "LCSC" "C2907044"
+			(at 118.11 85.09 90)
+			(hide yes)
+			(show_name no)

Commit message: (feat): routing v2
Connections:
- net D+: now reaches U1.3 (I/O2), USB_C1.A6 (D+), USB_C1.B6 (D+)
- net D-: now reaches U1.1 (I/O1), USB_C1.A7 (D-), USB_C1.B7 (D-)
Changed lines of the file:
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@@
+		)
+	)
+	(label "D+"
+		(at 107.95 92.71 0)
+		(effects
+			(font
+				(size 1.27 1.27)
+			)
+			(justify left bottom)
+		)
+	)
+	(label "D-"
+		(at 107.95 90.17 0)
+		(effects
+			(font
+				(size 1.27 1.27)
+			)
+			(justify left bottom)
 		)
 	)

Commit message: Updates to schematic by Ludo <3
Other:
- moved on the sheet: C18, R20, U1, USB1
