File: ControlBoard/io.kicad_sch (KiCad schematic)
At the start: 10 parts, among them U1 USBLC6-2P6

Commit message: (fixes): various small fixes
Parts:
- USB1: value LED -> GREEN
Changed lines of the file:
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@@
 		(in_pos_files yes)
 		(dnp no)
-		(fields_autoplaced yes)
 		(property "Reference" "USB1"
-			(at 67.31 90.4874 90)
+			(at 62.738 89.662 90)
 			(show_name no)
 			(do_not_autoplace no)
@@
 					(size 1.27 1.27)
 				)
-				(justify right)
+				(justify left)
 			)
 		)
-		(property "Value" "LED"
-			(at 67.31 93.0274 90)
+		(property "Value" "GREEN"
+			(at 62.23 91.694 90)
 			(show_name no)
 			(do_not_autoplace no)
@@
 					(size 1.27 1.27)
 				)
-				(justify right)
+				(justify left)
 			)
 		)

Commit message: (prod): final adjustements and final bom for production
Parts:
- UART1: footprint Connector_PinHeader_1.00mm:PinHeader_1x04_P1.00mm_Vertical -> Connector_PinHeader_2.54mm:PinHeader_1x04_P2.54mm_Vertical
- USB_C1: LCSC C3151746 -> C2765186
Changed lines of the file:
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@@
 			)
 		)
-		(property "Footprint" "Connector_PinHeader_1.00mm:PinHeader_1x04_P1.00mm_Vertical"
+		(property "Footprint" "Connector_PinHeader_2.54mm:PinHeader_1x04_P2.54mm_Vertical"
 			(at 179.07 88.9 0)
 			(hide yes)
@@
 			)
 		)
-		(property "LCSC" "C3151746"
+		(property "LCSC" "C2765186"
 			(at 137.16 92.71 0)
 			(hide yes)
