File: ControlBoard/CDFR2027-PAMIs-ELEC-control.kicad_sch (KiCad schematic)
At the start: 13 parts, among them SW1 Push_BOOT, SW2 Push_ENABLE, U1 ESP32-S3-WROOM-1

Commit message: WIP: placement
Parts:
- removed C12: TBD, Package_SO:SOIC-8_3.9x4.9mm_P1.27mm, symbol Device:C
- C1: renamed from C13; footprint (none) -> Capacitor_SMD:C_0603_1608Metric
- C2: renamed from C9; footprint Package_SO:SOIC-8_3.9x4.9mm_P1.27mm -> Capacitor_SMD:C_0603_1608Metric
- C3: renamed from C10; footprint Package_SO:SOIC-8_3.9x4.9mm_P1.27mm -> Capacitor_SMD:C_0603_1608Metric
- H1, H4: footprint (none) -> MountingHole:MountingHole_3.2mm_M3
- H2: renamed from H3; footprint (none) -> MountingHole:MountingHole_3.2mm_M3
- H3: renamed from H2; footprint (none) -> MountingHole:MountingHole_3.2mm_M3
- R1: renamed from R9; footprint (none) -> Resistor_SMD:R_0603_1608Metric
- R2: renamed from R8; value TBD -> 10k; footprint (none) -> Resistor_SMD:R_0603_1608Metric
- SW_BOOT1: renamed from SW1; footprint (none) -> Button_Switch_THT:SW_PUSH_6mm
- SW_ENABLE1: renamed from SW2; footprint (none) -> Button_Switch_THT:SW_PUSH_6mm
- renumbered U1 to ESP32-S3-WROOM1
Connections:
- net Actuators & Utility/SERVO_A renamed Actuators & Utility/SERVO_1
- net Actuators & Utility/SERVO_B renamed Actuators & Utility/SERVO_2
- net Actuators & Utility/SERVO_C renamed Actuators & Utility/SERVO_3
- net Actuators & Utility/SERVO_D renamed Actuators & Utility/SERVO_4
- net Motors/DC_A_IN1 renamed Motors/DC_1_IN1
- net Motors/DC_A_IN2 renamed Motors/DC_1_IN2
- net Motors/DC_B_IN1 renamed Motors/DC_2_IN1
- net Motors/DC_B_IN2 renamed Motors/DC_2_IN2
- net Motors/DC_C_IN1 renamed Motors/DC_3_IN1
- net Motors/DC_C_IN2 renamed Motors/DC_3_IN2
Other:
- sheet Actuators & Utility ports: added SERVO_1, SERVO_2, SERVO_3, SERVO_4; removed SERVO_A, SERVO_B, SERVO_C, SERVO_D
- sheet Motors ports: added DC_1_IN1, DC_1_IN2, DC_2_IN1, DC_2_IN2, DC_3_IN1, DC_3_IN2; removed DC_A_IN1, DC_A_IN2, DC_B_IN1, DC_B_IN2, DC_C_IN1, DC_C_IN2

Commit message: fix: a lot of small things, simplify
Parts:
- added R24, R25: 10k, Resistor_SMD:R_0201_0603Metric, symbol Device:R
- C2: value 0.22uF -> 22uF
Connections:
- net Actuators & Utility/IO10 is gone; now on net Actuators & Utility/SERVO_3: ESP32-S3-WROOM1.22 (IO14)
- net Actuators & Utility/LED_STRIP is gone; now on net Actuators & Utility/SERVO_4: ESP32-S3-WROOM1.8 (IO15)
- net Actuators & Utility/SERVO_3: no longer ESP32-S3-WROOM1.16 (IO46)
- net Actuators & Utility/SERVO_4: no longer ESP32-S3-WROOM1.26 (IO45)
- net GND: now also R24.2, R25.2
- net Actuators & Utility/IO11: no longer names the net of ESP32-S3-WROOM1.21 (IO13)
- net Actuators & Utility/IO12: no longer names the net of ESP32-S3-WROOM1.20 (IO12)
- net Actuators & Utility/IO13: no longer names the net of ESP32-S3-WROOM1.19 (IO11)
- net Actuators & Utility/IO14: no longer names the net of ESP32-S3-WROOM1.18 (IO10)
- new net: ESP32-S3-WROOM1.26 (IO45), R24.1
- new net: ESP32-S3-WROOM1.16 (IO46), R25.1
- no-connect marks 6 -> 10
Other:
- sheet Actuators & Utility ports: added none; removed IO10, IO11, IO12, IO13, IO14, LED_STRIP

Commit message: Routing V1 done
Parts:
- R2: footprint Resistor_SMD:R_0603_1608Metric -> Resistor_SMD:R_0805_2012Metric
- R24: footprint Resistor_SMD:R_0201_0603Metric -> PCM_SparkFun-Resistor:R_0603_1608Metric
- R25: footprint Resistor_SMD:R_0201_0603Metric -> Resistor_SMD:R_0603_1608Metric
Connections:
- net Actuators & Utility/SERVO_1: now also ESP32-S3-WROOM1.24 (IO47); no longer ESP32-S3-WROOM1.25 (IO48)
- net Actuators & Utility/SERVO_2: now also ESP32-S3-WROOM1.25 (IO48); no longer ESP32-S3-WROOM1.24 (IO47)
- net Actuators & Utility/GPIO4: now reaches ESP32-S3-WROOM1.18 (IO10)
- net Actuators & Utility/GPIO3: now reaches ESP32-S3-WROOM1.19 (IO11)
- net Actuators & Utility/GPIO2: now reaches ESP32-S3-WROOM1.20 (IO12)
- net Actuators & Utility/GPIO1: now reaches ESP32-S3-WROOM1.21 (IO13)
- no-connect marks 10 -> 6
Other:
- sheet Actuators & Utility ports: added GPIO1, GPIO2, GPIO3, GPIO4; removed none
Changed lines of the file:
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@@
-	)
-	(no_connect
-		(at 138.43 96.52)
-	)
-	(no_connect
-		(at 138.43 101.6)
-	)
-	(no_connect
-		(at 138.43 104.14)
 	)
 	(no_connect
@@
 	)
 	(no_connect
-		(at 138.43 99.06)
-	)
-	(no_connect
 		(at 168.91 83.82)
 	)
@@
 	(wire
 		(pts
-			(xy 171.45 111.76) (xy 171.45 130.81)
+			(xy 129.54 130.81) (xy 129.54 104.14)
 		)
 		(stroke
@@
 	(wire
 		(pts
-			(xy 173.99 109.22) (xy 173.99 130.81)
-		)
-		(stroke
-			(width 0)
-			(type default)
-		)
-	)
-	(wire
-		(pts
 			(xy 138.43 83.82) (xy 91.44 83.82)
 		)
@@
 	(wire
 		(pts
+			(xy 127 130.81) (xy 127 101.6)
+		)
+		(stroke
+			(width 0)
+			(type default)
+		)
+	)
+	(wire
+		(pts
 			(xy 105.41 36.83) (xy 105.41 46.99)
 		)
@@
 	(wire
 		(pts
+			(xy 121.92 96.52) (xy 121.92 130.81)
+		)
+		(stroke
+			(width 0)
+			(type default)
+		)
+	)
+	(wire
+		(pts
 			(xy 180.34 104.14) (xy 182.88 104.14)
 		)
@@
 	(wire
 		(pts
-			(xy 168.91 109.22) (xy 173.99 109.22)
+			(xy 168.91 109.22) (xy 175.26 109.22)
 		)
 		(stroke
@@
 	(wire
 		(pts
-			(xy 168.91 111.76) (xy 171.45 111.76)
+			(xy 168.91 111.76) (xy 172.72 111.76)
 		)
 		(stroke
@@
 	(wire
 		(pts
+			(xy 172.72 130.81) (xy 172.72 111.76)
+		)
+		(stroke
+			(width 0)
+			(type default)
+		)
+	)
+	(wire
+		(pts
 			(xy 168.91 71.12) (xy 196.85 71.12)
 		)
@@
 	(wire
 		(pts
+			(xy 129.54 104.14) (xy 138.43 104.14)
+		)
+		(stroke
+			(width 0)
+			(type default)
+		)
+	)
+	(wire
+		(pts
 			(xy 168.91 78.74) (xy 196.85 78.74)
 		)
@@
 	(wire
 		(pts
+			(xy 175.26 109.22) (xy 175.26 130.81)
+		)
+		(stroke
+			(width 0)
+			(type default)
+		)
+	)
+	(wire
+		(pts
 			(xy 132.08 59.69) (xy 132.08 66.04)
 		)
@@
 	(wire
 		(pts
+			(xy 124.46 99.06) (xy 138.43 99.06)
+		)
+		(stroke
+			(width 0)
+			(type default)
+		)
+	)
+	(wire
+		(pts
 			(xy 182.88 104.14) (xy 185.42 104.14)
 		)
@@
 	(wire
 		(pts
+			(xy 127 101.6) (xy 138.43 101.6)
+		)
+		(stroke
+			(width 0)
+			(type default)
+		)
+	)
+	(wire
+		(pts
 			(xy 147.32 48.26) (xy 153.67 48.26)
 		)
@@
 	(wire
 		(pts
+			(xy 138.43 96.52) (xy 121.92 96.52)
+		)
+		(stroke
+			(width 0)
+			(type default)
+		)
+	)
+	(wire
+		(pts
 			(xy 168.91 93.98) (xy 196.85 93.98)
 		)
@@
 		(pts
 			(xy 129.54 71.12) (xy 138.43 71.12)
+		)
+		(stroke
+			(width 0)
+			(type default)
+		)
+	)
+	(wire
+		(pts
+			(xy 124.46 130.81) (xy 124.46 99.06)
 		)
 		(stroke
@@
 			)
 		)
-		(property "Footprint" "Resistor_SMD:R_0201_0603Metric"
+		(property "Footprint" "PCM_SparkFun-Resistor:R_0603_1608Metric"
 			(at 176.53 105.918 90)
 			(hide yes)
@@
 			)
 		)
-		(property "Footprint" "Resistor_SMD:R_0201_0603Metric"
+		(property "Footprint" "Resistor_SMD:R_0603_1608Metric"
 			(at 176.53 108.458 90)
 			(hide yes)
@@
 			)
 		)
-		(property "Footprint" "Resistor_SMD:R_0603_1608Metric"
+		(property "Footprint" "Resistor_SMD:R_0805_2012Metric"
 			(at 143.51 57.912 90)
 			(hide yes)
@@
 		)
 		(property "Value" "GND"
-			(at 93.98 36.8299 90)
-			(show_name no)
-			(do_not_autoplace no)
-			(effects
-				(font
-					(size 1.27 1.27)
-				)
-				(justify right)
+			(at 96.52 33.02 90)
+			(show_name no)
+			(do_not_autoplace no)
+			(effects
+				(font
+					(size 1.27 1.27)
+				)
 			)
 		)
@@
 		)
 		(pin "SERVO_1" input
-			(at 171.45 130.81 90)
+			(at 175.26 130.81 90)
 			(effects
 				(font
@@
 		)
 		(pin "SERVO_2" input
-			(at 173.99 130.81 90)
+			(at 172.72 130.81 90)
 			(effects
 				(font
@@
 			(effects
 				(font
+					(size 1.27 1.27)
+				)
+				(justify right)
+			)
+		)
+		(pin "GPIO1" input
+			(at 129.54 130.81 90)
+			(effects
+				(font
+					(size 1.27 1.27)
+				)
+				(justify right)
+			)
+		)
+		(pin "GPIO2" input
+			(at 127 130.81 90)
+			(effects
+				(font
+					(size 1.27 1.27)
+				)
+				(justify right)
+			)
+		)
+		(pin "GPIO3" input
+			(at 124.46 130.81 90)
+			(effects
+				(font
+					(size 1.27 1.27)
+				)
+				(justify right)
+			)
+		)
+		(pin "GPIO4" input
+			(at 121.92 130.81 90)
+			(effects
+				(font

Commit message: text
Connections:
- net Actuators & Utility/GPIO1 renamed Actuators & Utility/GPIO13
- net Actuators & Utility/GPIO2 renamed Actuators & Utility/GPIO12
- net Actuators & Utility/GPIO3 renamed Actuators & Utility/GPIO11
- net Actuators & Utility/GPIO4 renamed Actuators & Utility/GPIO10
Other:
- sheet Actuators & Utility ports: added GPIO10, GPIO11, GPIO12, GPIO13; removed GPIO1, GPIO2, GPIO3, GPIO4
Changed lines of the file:
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@@
 			)
 		)
-		(pin "GPIO1" input
+		(pin "GPIO13" input
 			(at 129.54 130.81 90)
 			(effects
@@
 			)
 		)
-		(pin "GPIO2" input
+		(pin "GPIO12" input
 			(at 127 130.81 90)
 			(effects
@@
 			)
 		)
-		(pin "GPIO3" input
+		(pin "GPIO11" input
 			(at 124.46 130.81 90)
 			(effects
@@
 			)
 		)
-		(pin "GPIO4" input
+		(pin "GPIO10" input
 			(at 121.92 130.81 90)
 			(effects

Commit message: (feat): bom
Parts:
- C1, C3: LCSC (none) -> C1591
- C2: LCSC (none) -> C59461
- ESP32-S3-WROOM1: LCSC (none) -> C3013946
- R1: LCSC (none) -> C22548
- R2, R24, R25: LCSC (none) -> C84376
Changed lines of the file:
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@@
+			)
+		)
+		(property "LCSC" "C1591"
+			(at 113.03 46.99 90)
+			(hide yes)
+			(show_name no)
+			(do_not_autoplace no)
+			(effects
+				(font
+					(size 1.27 1.27)
+				)
 			)
 		)
@@
 			)
 		)
+		(property "LCSC" "C22548"
+			(at 125.73 59.69 90)
+			(hide yes)
+			(show_name no)
+			(do_not_autoplace no)
+			(effects
+				(font
+					(size 1.27 1.27)
+				)
+			)
+		)
 		(pin "1"
 		)
@@
 			)
 		)
+		(property "LCSC" "C1591"
+			(at 143.51 48.26 90)
+			(hide yes)
+			(show_name no)
+			(do_not_autoplace no)
+			(effects
+				(font
+					(size 1.27 1.27)
+				)
+			)
+		)
 		(pin "2"
 		)
@@
 		(property "Description" "Resistor"
 			(at 176.53 104.14 0)
+			(hide yes)
+			(show_name no)
+			(do_not_autoplace no)
+			(effects
+				(font
+					(size 1.27 1.27)
+				)
+			)
+		)
+		(property "LCSC" "C84376"
+			(at 176.53 104.14 90)
 			(hide yes)
 			(show_name no)
@@
 			)
 		)
+		(property "LCSC" "C84376"
+			(at 176.53 106.68 90)
+			(hide yes)
+			(show_name no)
+			(do_not_autoplace no)
+			(effects
+				(font
+					(size 1.27 1.27)
+				)
+			)
+		)
 		(pin "1"
 		)
@@
 			)
 		)
+		(property "LCSC" "C84376"
+			(at 143.51 59.69 90)
+			(hide yes)
+			(show_name no)
+			(do_not_autoplace no)
+			(effects
+				(font
+					(size 1.27 1.27)
+				)
+			)
+		)
 		(pin "2"
 		)
@@
 			)
 		)
+		(property "LCSC" "C59461"
+			(at 143.51 36.83 90)
+			(hide yes)
+			(show_name no)
+			(do_not_autoplace no)
+			(effects
+				(font
+					(size 1.27 1.27)
+				)
+			)
+		)
 		(pin "2"
 		)
@@
 			(at 153.67 88.9 0)
 			(hide yes)
+			(show_name no)
+			(do_not_autoplace no)
+			(effects
+				(font
+					(size 1.27 1.27)
+				)
+			)
+		)
+		(property "LCSC" "C3013946"
+			(at 153.67 88.9 0)
+			(hide yes)

Commit message: Updates to schematic by Ludo <3
Connections:
- net EN: now reaches ESP32-S3-WROOM1.3 (EN), R1.2, R2.2
- net BOOT: now reaches ESP32-S3-WROOM1.27 (IO0), SW_BOOT1.2
Other:
- moved on the sheet: C3

Commit message: (fixes): various small fixes
Parts:
- SW_BOOT1, SW_ENABLE1: LCSC (none) -> C49234152
Other:
- moved on the sheet: C1, R1, R2, SW_BOOT1, SW_ENABLE1

Commit message: (prod): final adjustements and final bom for production
Parts:
- SW_BOOT1, SW_ENABLE1: LCSC C49234152 -> C55271357
Connections:
- net Actuators & Utility/GPIO10: no longer names the net of ESP32-S3-WROOM1.18 (IO10)
- net Actuators & Utility/GPIO11: no longer names the net of ESP32-S3-WROOM1.19 (IO11)
- net Actuators & Utility/GPIO12: no longer names the net of ESP32-S3-WROOM1.20 (IO12)
- net Actuators & Utility/GPIO13: no longer names the net of ESP32-S3-WROOM1.21 (IO13)
- no-connect marks 6 -> 10
Other:
- sheet Actuators & Utility ports: added none; removed GPIO10, GPIO11, GPIO12, GPIO13
Changed lines of the file:
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@@
+	)
+	(no_connect
+		(at 138.43 101.6)
+	)
+	(no_connect
+		(at 138.43 96.52)
 	)
 	(no_connect
@@
 	)
 	(no_connect
+		(at 138.43 99.06)
+	)
+	(no_connect
 		(at 168.91 86.36)
 	)
@@
 	)
 	(no_connect
+		(at 138.43 104.14)
+	)
+	(no_connect
 		(at 168.91 83.82)
 	)
@@
 	(wire
 		(pts
-			(xy 127 101.6) (xy 138.43 101.6)
-		)
-		(stroke
-			(width 0)
-			(type default)
-		)
-	)
-	(wire
-		(pts
 			(xy 170.18 41.91) (xy 170.18 45.72)
 		)
@@
 	(wire
 		(pts
-			(xy 102.87 115.57) (xy 121.92 115.57)
-		)
-		(stroke
-			(width 0)
-			(type default)
-		)
-	)
-	(wire
-		(pts
 			(xy 121.92 58.42) (xy 121.92 57.15)
 		)
@@
 	(wire
 		(pts
-			(xy 127 120.65) (xy 127 101.6)
-		)
-		(stroke
-			(width 0)
-			(type default)
-		)
-	)
-	(wire
-		(pts
 			(xy 180.34 104.14) (xy 182.88 104.14)
 		)
@@
 	(wire
 		(pts
-			(xy 138.43 99.06) (xy 124.46 99.06)
-		)
-		(stroke
-			(width 0)
-			(type default)
-		)
-	)
-	(wire
-		(pts
 			(xy 102.87 130.81) (xy 137.16 130.81)
 		)
@@
 	(wire
 		(pts
-			(xy 124.46 118.11) (xy 102.87 118.11)
-		)
-		(stroke
-			(width 0)
-			(type default)
-		)
-	)
-	(wire
-		(pts
 			(xy 102.87 93.98) (xy 111.76 93.98)
 		)
@@
 	(wire
 		(pts
-			(xy 129.54 123.19) (xy 102.87 123.19)
-		)
-		(stroke
-			(width 0)
-			(type default)
-		)
-	)
-	(wire
-		(pts
 			(xy 102.87 96.52) (xy 114.3 96.52)
 		)
@@
 	(wire
 		(pts
-			(xy 102.87 120.65) (xy 127 120.65)
-		)
-		(stroke
-			(width 0)
-			(type default)
-		)
-	)
-	(wire
-		(pts
 			(xy 134.62 109.22) (xy 134.62 128.27)
 		)
@@
 	(wire
 		(pts
-			(xy 121.92 96.52) (xy 138.43 96.52)
-		)
-		(stroke
-			(width 0)
-			(type default)
-		)
-	)
-	(wire
-		(pts
 			(xy 168.91 78.74) (xy 196.85 78.74)
 		)
@@
 	(wire
 		(pts
-			(xy 124.46 99.06) (xy 124.46 118.11)
-		)
-		(stroke
-			(width 0)
-			(type default)
-		)
-	)
-	(wire
-		(pts
-			(xy 129.54 104.14) (xy 129.54 123.19)
-		)
-		(stroke
-			(width 0)
-			(type default)
-		)
-	)
-	(wire
-		(pts
 			(xy 101.6 45.72) (xy 101.6 46.99)
 		)
@@
 	(wire
 		(pts
-			(xy 138.43 104.14) (xy 129.54 104.14)
-		)
-		(stroke
-			(width 0)
-			(type default)
-		)
-	)
-	(wire
-		(pts
 			(xy 102.87 101.6) (xy 116.84 101.6)
 		)
@@
 		(pts
 			(xy 153.67 41.91) (xy 157.48 41.91)
-		)
-		(stroke
-			(width 0)
-			(type default)
-		)
-	)
-	(wire
-		(pts
-			(xy 121.92 115.57) (xy 121.92 96.52)
 		)
 		(stroke
@@
 				(font
 					(size 1.27 1.27)
+					(thickness 0.1588)
 				)
 				(justify right)
@@
 			)
 		)
-		(property "LCSC" "C49234152"
+		(property "LCSC" "C55271357"
 			(at 101.6 52.07 90)
 			(hide yes)
@@
 			)
 		)
-		(property "LCSC" "C49234152"
+		(property "LCSC" "C55271357"
 			(at 121.92 52.07 90)
 			(hide yes)
@@
 			(effects
 				(font
-					(size 1.27 1.27)
-				)
-				(justify right)
-			)
-		)
-		(pin "GPIO13" input
-			(at 102.87 123.19 0)
-			(effects
-				(font
-					(size 1.27 1.27)
-				)
-				(justify right)
-			)
-		)
-		(pin "GPIO12" input
-			(at 102.87 120.65 0)
-			(effects
-				(font
-					(size 1.27 1.27)
-				)
-				(justify right)
-			)
-		)
-		(pin "GPIO11" input
-			(at 102.87 118.11 0)
-			(effects
-				(font
-					(size 1.27 1.27)
-				)
-				(justify right)
-			)
-		)
-		(pin "GPIO10" input
-			(at 102.87 115.57 0)
-			(effects
-				(font
