File: ControlBoard/motors.kicad_sch (KiCad schematic)
At the start: 21 parts, among them U4 DRV8871DDA, U6 DRV8871DDA, U7 DRV8871DDA

Commit message: WIP: placement
Parts:
- Pin_DC_OUT_1: renamed from Pin_DC_OUT_A; footprint (none) -> Connector_JST:JST_XH_B2B-XH-A_1x02_P2.50mm_Vertical
- Pin_DC_OUT_2: renamed from Pin_DC_OUT_B; footprint (none) -> Connector_JST:JST_XH_B2B-XH-A_1x02_P2.50mm_Vertical
- Pin_DC_OUT_3: renamed from Pin_DC_OUT_C; footprint (none) -> Connector_JST:JST_XH_B2B-XH-A_1x02_P2.50mm_Vertical
- renumbered C14 to C12, C16 to C13, C15 to C14, C17 to C15, C18 to C16, C20 to C17, U4 to DC_DRIVER1, U6 to DC_DRIVER2, U7 to DC_DRIVER3, R18 to R10, R19 to R11, R15 to R12, R16 to R13, R20 to R15, R21 to R16, R22 to R17, R17 to R9
Connections:
- net DC_A_IN1 renamed DC_1_IN1
- net DC_A_IN2 renamed DC_1_IN2
- net DC_B_IN1 renamed DC_2_IN1
- net DC_B_IN2 renamed DC_2_IN2
- net DC_C_IN1 renamed DC_3_IN1
- net DC_C_IN2 renamed DC_3_IN2

Commit message: Routing V1 done
Parts:
- renumbered Pin_DC_OUT_1 to DC_OUT_1, Pin_DC_OUT_2 to DC_OUT_2, Pin_DC_OUT_3 to DC_OUT_3

Commit message: (feat): bom
Parts:
- DC_OUT_1, DC_OUT_2, DC_OUT_3: LCSC (none) -> C158012
Changed lines of the file:
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@@
+			)
+		)
+		(property "LCSC" "C158012"
+			(at 260.35 90.17 0)
+			(hide yes)
+			(show_name no)
+			(do_not_autoplace no)
+			(effects
+				(font
+					(size 1.27 1.27)
+				)
 			)
 		)
@@
 			)
 		)
+		(property "LCSC" "C158012"
+			(at 83.82 90.17 0)
+			(hide yes)
+			(show_name no)
+			(do_not_autoplace no)
+			(effects
+				(font
+					(size 1.27 1.27)
+				)
+			)
+		)
 		(pin "2"
 		)
@@
 			(at 170.18 90.17 0)
 			(hide yes)
+			(show_name no)
+			(do_not_autoplace no)
+			(effects
+				(font
+					(size 1.27 1.27)
+				)
+			)
+		)
+		(property "LCSC" "C158012"
+			(at 170.18 90.17 0)
+			(hide yes)

Commit message: (feat): routing v2
Parts:
- C13, C15, C17: footprint Capacitor_SMD:C_0603_1608Metric -> Capacitor_SMD:C_0805_2012Metric; LCSC C1591 -> C49678
- R10, R12, R13, R15, R16, R9: footprint Resistor_SMD:R_0603_1608Metric -> Resistor_SMD:R_0805_2012Metric; LCSC C98220 -> C17414
- R11, R14, R17: footprint Resistor_SMD:R_0603_1608Metric -> Resistor_SMD:R_0805_2012Metric; LCSC C2930081 -> C2907246
Changed lines of the file:
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@@
 			)
 		)
-		(property "Footprint" "Resistor_SMD:R_0603_1608Metric"
+		(property "Footprint" "Resistor_SMD:R_0805_2012Metric"
 			(at 160.528 104.14 90)
 			(hide yes)
@@
 			)
 		)
-		(property "LCSC" "C2930081"
+		(property "LCSC" "C2907246"
 			(at 158.75 104.14 0)
 			(hide yes)
@@
 			)
 		)
-		(property "Footprint" "Resistor_SMD:R_0603_1608Metric"
+		(property "Footprint" "Resistor_SMD:R_0805_2012Metric"
 			(at 131.572 101.6 90)
 			(hide yes)
@@
 			)
 		)
-		(property "LCSC" "C98220"
+		(property "LCSC" "C17414"
 			(at 133.35 101.6 0)
 			(hide yes)
@@
 			)
 		)
-		(property "Footprint" "Capacitor_SMD:C_0603_1608Metric"
+		(property "Footprint" "Capacitor_SMD:C_0805_2012Metric"
 			(at 168.6052 78.74 0)
 			(hide yes)
@@
 			)
 		)
-		(property "LCSC" "C1591"
+		(property "LCSC" "C49678"
 			(at 167.64 74.93 90)
 			(hide yes)
@@
 			)
 		)
-		(property "Footprint" "Resistor_SMD:R_0603_1608Metric"
+		(property "Footprint" "Resistor_SMD:R_0805_2012Metric"
 			(at 122.682 101.6 90)
 			(hide yes)
@@
 			)
 		)
-		(property "LCSC" "C98220"
+		(property "LCSC" "C17414"
 			(at 124.46 101.6 0)
 			(hide yes)
@@
 			)
 		)
-		(property "Footprint" "Capacitor_SMD:C_0603_1608Metric"
+		(property "Footprint" "Capacitor_SMD:C_0805_2012Metric"
 			(at 256.2352 78.74 0)
 			(hide yes)
@@
 			)
 		)
-		(property "LCSC" "C1591"
+		(property "LCSC" "C49678"
 			(at 255.27 74.93 90)
 			(hide yes)
@@
 			)
 		)
-		(property "Footprint" "Resistor_SMD:R_0603_1608Metric"
+		(property "Footprint" "Resistor_SMD:R_0805_2012Metric"
 			(at 74.168 104.14 90)
 			(hide yes)
@@
 			)
 		)
-		(property "LCSC" "C2930081"
+		(property "LCSC" "C2907246"
 			(at 72.39 104.14 0)
 			(hide yes)
@@
 			)
 		)
-		(property "Footprint" "Resistor_SMD:R_0603_1608Metric"
+		(property "Footprint" "Resistor_SMD:R_0805_2012Metric"
 			(at 248.158 104.14 90)
 			(hide yes)
@@
 			)
 		)
-		(property "LCSC" "C2930081"
+		(property "LCSC" "C2907246"
 			(at 246.38 104.14 0)
 			(hide yes)
@@
 			)
 		)
-		(property "Footprint" "Resistor_SMD:R_0603_1608Metric"
+		(property "Footprint" "Resistor_SMD:R_0805_2012Metric"
 			(at 219.202 101.6 90)
 			(hide yes)
@@
 			)
 		)
-		(property "LCSC" "C98220"
+		(property "LCSC" "C17414"
 			(at 220.98 101.6 0)
 			(hide yes)
@@
 			)
 		)
-		(property "Footprint" "Capacitor_SMD:C_0603_1608Metric"
+		(property "Footprint" "Capacitor_SMD:C_0805_2012Metric"
 			(at 80.9752 80.01 0)
 			(hide yes)
@@
 			)
 		)
-		(property "LCSC" "C1591"
+		(property "LCSC" "C49678"
 			(at 80.01 76.2 90)
 			(hide yes)
@@
 			)
 		)
-		(property "Footprint" "Resistor_SMD:R_0603_1608Metric"
+		(property "Footprint" "Resistor_SMD:R_0805_2012Metric"
 			(at 45.212 101.6 90)
 			(hide yes)
@@
 			)
 		)
-		(property "LCSC" "C98220"
+		(property "LCSC" "C17414"
 			(at 46.99 101.6 0)
 			(hide yes)
@@
 			)
 		)
-		(property "Footprint" "Resistor_SMD:R_0603_1608Metric"
+		(property "Footprint" "Resistor_SMD:R_0805_2012Metric"
 			(at 210.312 101.6 90)
 			(hide yes)
@@
 			)
 		)
-		(property "LCSC" "C98220"
+		(property "LCSC" "C17414"
 			(at 212.09 101.6 0)
 			(hide yes)
@@
 			)
 		)
-		(property "Footprint" "Resistor_SMD:R_0603_1608Metric"
+		(property "Footprint" "Resistor_SMD:R_0805_2012Metric"
 			(at 36.322 101.6 90)
 			(hide yes)
@@
 			)
 		)
-		(property "LCSC" "C98220"
+		(property "LCSC" "C17414"
 			(at 38.1 101.6 0)
 			(hide yes)

Commit message: Updates to schematic by Ludo <3
Changed lines of the file:
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@@
 		(property "Value" "GND"
 			(at 258.064 78.486 0)
+			(hide yes)
 			(show_name no)
 			(do_not_autoplace no)
@@
 		(property "Value" "GND"
 			(at 62.23 113.792 0)
+			(hide yes)
 			(show_name no)
 			(do_not_autoplace no)
@@
 		(property "Value" "GND"
 			(at 148.59 113.792 0)
+			(hide yes)
 			(show_name no)
 			(do_not_autoplace no)
@@
 		(property "Value" "GND"
 			(at 170.434 78.486 0)
+			(hide yes)
 			(show_name no)
 			(do_not_autoplace no)
@@
 		(property "Value" "GND"
 			(at 236.22 113.792 0)
+			(hide yes)
 			(show_name no)
 			(do_not_autoplace no)
@@
 		(property "Value" "GND"
 			(at 71.374 79.756 0)
+			(hide yes)
 			(show_name no)
 			(do_not_autoplace no)
@@
 		(property "Value" "GND"
 			(at 246.634 78.486 0)
+			(hide yes)
 			(show_name no)
 			(do_not_autoplace no)
@@
 		(property "Value" "GND"
 			(at 82.804 79.756 0)
+			(hide yes)
 			(show_name no)
 			(do_not_autoplace no)
@@
 		(property "Value" "GND"
 			(at 159.004 78.486 0)
-			(show_name no)
-			(do_not_autoplace no)
+			(hide yes)
+			(show_name no)
+			(do_not_autoplace no)

Commit message: (prod): final adjustements and final bom for production
Parts:
- C12: LCSC C128464 -> C128464
- DC_DRIVER1, DC_DRIVER2, DC_DRIVER3: LCSC C701805 -> C75864
Changed lines of the file:
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@@
 			)
 		)
-		(property "LCSC" "C128464"
+		(property "LCSC" " C128464 "
 			(at 68.58 76.2 90)
 			(hide yes)
@@
 			)
 		)
-		(property "LCSC" "C701805"
+		(property "LCSC" " C75864 "
 			(at 236.22 95.25 0)
 			(hide yes)
@@
 			)
 		)
-		(property "LCSC" "C701805"
+		(property "LCSC" " C75864 "
 			(at 62.23 95.25 0)
 			(hide yes)
@@
 			)
 		)
-		(property "LCSC" "C701805"
+		(property "LCSC" " C75864 "
 			(at 148.59 95.25 0)
 			(hide yes)
