File: ControlBoard/power.kicad_sch (KiCad schematic)
At the start: 34 parts, among them Q1 PMOS

Commit message: (fixes): various small fixes
Parts:
- LED_3.3V1, LED_5V1, LED_BATT1: value LED -> RED
Changed lines of the file:
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@@
 			)
 		)
-		(property "Value" "LED"
+		(property "Value" "RED"
 			(at 128.27 127.3174 90)
 			(show_name no)
@@
 			)
 		)
-		(property "Value" "LED"
+		(property "Value" "RED"
 			(at 95.25 127.3174 90)
 			(show_name no)
@@
 			)
 		)
-		(property "Value" "LED"
+		(property "Value" "RED"
 			(at 113.03 127 90)
 			(show_name no)

Commit message: (prod): final adjustements and final bom for production
Parts:
- BAU1, C_BATT1: LCSC C32713268 -> C99102
- C5: LCSC C2163886 -> C48935390
- L1: LCSC C5349706 -> C340380
- R6: LCSC C4045076 -> C441882
Changed lines of the file:
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@@
 			)
 		)
-		(property "LCSC" "C4045076"
+		(property "LCSC" "C441882"
 			(at 91.44 116.84 0)
 			(hide yes)
@@
 			)
 		)
-		(property "LCSC" "C32713268"
+		(property "LCSC" "C99102"
 			(at 29.21 64.77 0)
 			(hide yes)
@@
 			)
 		)
-		(property "LCSC" "C32713268"
+		(property "LCSC" "C99102"
 			(at 48.26 59.69 90)
 			(hide yes)
@@
 			)
 		)
-		(property "LCSC" "C5349706"
+		(property "LCSC" "C340380"
 			(at 154.94 67.31 90)
 			(hide yes)
@@
 			)
 		)
-		(property "LCSC" "C2163886"
+		(property "LCSC" " C48935390 "
 			(at 87.63 74.93 0)
 			(hide yes)
